File: hardware/gizmo.kicad_sch (KiCad schematic)
At the start: 22 parts, among them J2 USB4505-03-0-A, U1 MPM3606AGQV-P, U2 ESP32-C3-MINI-1, U3 CAT24M01Y, U5 CY8CMBR3108

Commit message: Hook up eeprom and capsense ic
Parts:
- added C25, C27: 0.1uF, Capacitor_SMD:C_0603_1608Metric, symbol Device:C_Small
- added C26: 2.2nF 5V X7R, symbol Device:C_Small
Connections:
- net +3.3V: now also U5.5 (VDDIO), U5.6 (VDD), C27.1
- net GND: now also U5.17 (EP), U5.7 (VSS), C25.2, C26.2, C27.2
- net CAPSENSE_INT: now reaches U2.21 (GPIO7)
- net CAPSENSE_INT: now also U5.16 (~{HI})
- net at U5.3 (CMOD): now also C26.1
- net at U5.4 (VCC): now also C25.1
- net LEDs/CI: no longer names the net of U2.6 (GPIO3/ADC1_CH3)
- net LEDs/DI: no longer names the net of U2.18 (GPIO4/ADC1_CH4)
- net U0_RX renamed LED_DATA
- net U0_TX renamed LED_CLK
- no-connect marks 8 -> 9
Other:
- note added: "0x37"
- note added: "0x50"
- note removed: "IO9 and IO2 must be high for SPI boot IO9 has internal weak pull up ADC inputs max out at 2.5V!"
- moved on the sheet: C1, C10, C2, C4, R1, R3, R7, R8, U2, U3, U5
